File: pcb/breadled.kicad_pcb (KiCad board)
At the start: 2 copper layers, 10.2 x 7.6 mm, 4 parts, among them J1 Conn_01x03_Male, J2 Conn_01x03_Male

Commit message: Add files via upload
Routing:
- net /GND: track 0.13 -> 9.99 mm
Other:
- board text added: "breadled v0.2.1"
- board text removed: "breadled v0.2"
Changed lines of the file:
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@@
     (thickness 1.6)
     (drawings 6)
-    (tracks 11)
+    (tracks 14)
     (zones 0)
     (modules 4)
@@
     (uvia_dia 0.3)
     (uvia_drill 0.1)
-    (add_net /5V)
-    (add_net /GND)
   )
   (net_class chonk ""
@@
     (uvia_dia 0.3)
     (uvia_drill 0.1)
+    (add_net /5V)
+    (add_net /GND)
     (add_net "Net-(D1-Pad2)")
     (add_net "Net-(D1-Pad4)")
@@
       (effects (font (size 1 1) (thickness 0.15)) (justify mirror))
     )
+    (fp_line (start 1.65 -0.73) (end -1.65 -0.73) (layer B.CrtYd) (width 0.05))
+    (fp_line (start 1.65 0.73) (end 1.65 -0.73) (layer B.CrtYd) (width 0.05))
+    (fp_line (start -1.65 0.73) (end 1.65 0.73) (layer B.CrtYd) (width 0.05))
+    (fp_line (start -1.65 -0.73) (end -1.65 0.73) (layer B.CrtYd) (width 0.05))
+    (fp_line (start -0.146267 -0.51) (end 0.146267 -0.51) (layer B.SilkS) (width 0.12))
+    (fp_line (start -0.146267 0.51) (end 0.146267 0.51) (layer B.SilkS) (width 0.12))
+    (fp_line (start 0.8 -0.4) (end -0.8 -0.4) (layer B.Fab) (width 0.1))
+    (fp_line (start 0.8 0.4) (end 0.8 -0.4) (layer B.Fab) (width 0.1))
+    (fp_line (start -0.8 0.4) (end 0.8 0.4) (layer B.Fab) (width 0.1))
     (fp_line (start -0.8 -0.4) (end -0.8 0.4) (layer B.Fab) (width 0.1))
-    (fp_line (start -0.8 0.4) (end 0.8 0.4) (layer B.Fab) (width 0.1))
-    (fp_line (start 0.8 0.4) (end 0.8 -0.4) (layer B.Fab) (width 0.1))
-    (fp_line (start 0.8 -0.4) (end -0.8 -0.4) (layer B.Fab) (width 0.1))
-    (fp_line (start -0.146267 0.51) (end 0.146267 0.51) (layer B.SilkS) (width 0.12))
-    (fp_line (start -0.146267 -0.51) (end 0.146267 -0.51) (layer B.SilkS) (width 0.12))
-    (fp_line (start -1.65 -0.73) (end -1.65 0.73) (layer B.CrtYd) (width 0.05))
-    (fp_line (start -1.65 0.73) (end 1.65 0.73) (layer B.CrtYd) (width 0.05))
-    (fp_line (start 1.65 0.73) (end 1.65 -0.73) (layer B.CrtYd) (width 0.05))
-    (fp_line (start 1.65 -0.73) (end -1.65 -0.73) (layer B.CrtYd) (width 0.05))
     (fp_text user %R (at 0 0 90) (layer B.Fab)
       (effects (font (size 0.4 0.4) (thickness 0.06)) (justify mirror))
@@
       (effects (font (size 1 1) (thickness 0.15)))
     )
+    (fp_circle (center 0 0) (end 0 -2) (layer F.Fab) (width 0.1))
+    (fp_line (start 3.65 2.75) (end 3.65 1.6) (layer F.SilkS) (width 0.12))
+    (fp_line (start -3.65 2.75) (end 3.65 2.75) (layer F.SilkS) (width 0.12))
+    (fp_line (start -3.65 -2.75) (end 3.65 -2.75) (layer F.SilkS) (width 0.12))
+    (fp_line (start 2.5 -2.5) (end -2.5 -2.5) (layer F.Fab) (width 0.1))
+    (fp_line (start 2.5 2.5) (end 2.5 -2.5) (layer F.Fab) (width 0.1))
+    (fp_line (start -2.5 2.5) (end 2.5 2.5) (layer F.Fab) (width 0.1))
+    (fp_line (start -2.5 -2.5) (end -2.5 2.5) (layer F.Fab) (width 0.1))
+    (fp_line (start 2.5 1.5) (end 1.5 2.5) (layer F.Fab) (width 0.1))
+    (fp_line (start -3.45 -2.75) (end -3.45 2.75) (layer F.CrtYd) (width 0.05))
+    (fp_line (start -3.45 2.75) (end 3.45 2.75) (layer F.CrtYd) (width 0.05))
+    (fp_line (start 3.45 2.75) (end 3.45 -2.75) (layer F.CrtYd) (width 0.05))
     (fp_line (start 3.45 -2.75) (end -3.45 -2.75) (layer F.CrtYd) (width 0.05))
-    (fp_line (start 3.45 2.75) (end 3.45 -2.75) (layer F.CrtYd) (width 0.05))
-    (fp_line (start -3.45 2.75) (end 3.45 2.75) (layer F.CrtYd) (width 0.05))
-    (fp_line (start -3.45 -2.75) (end -3.45 2.75) (layer F.CrtYd) (width 0.05))
-    (fp_line (start 2.5 1.5) (end 1.5 2.5) (layer F.Fab) (width 0.1))
-    (fp_line (start -2.5 -2.5) (end -2.5 2.5) (layer F.Fab) (width 0.1))
-    (fp_line (start -2.5 2.5) (end 2.5 2.5) (layer F.Fab) (width 0.1))
-    (fp_line (start 2.5 2.5) (end 2.5 -2.5) (layer F.Fab) (width 0.1))
-    (fp_line (start 2.5 -2.5) (end -2.5 -2.5) (layer F.Fab) (width 0.1))
-    (fp_line (start -3.65 -2.75) (end 3.65 -2.75) (layer F.SilkS) (width 0.12))
-    (fp_line (start -3.65 2.75) (end 3.65 2.75) (layer F.SilkS) (width 0.12))
-    (fp_line (start 3.65 2.75) (end 3.65 1.6) (layer F.SilkS) (width 0.12))
-    (fp_circle (center 0 0) (end 0 -2) (layer F.Fab) (width 0.1))
     (fp_text user 1 (at -4.15 -1.6 90) (layer F.SilkS) hide
       (effects (font (size 1 1) (thickness 0.15)))
@@
       (effects (font (size 1 1) (thickness 0.15)) (justify mirror))
     )
+    (fp_line (start 1.8 1.8) (end -1.8 1.8) (layer B.CrtYd) (width 0.05))
+    (fp_line (start 1.8 -6.85) (end 1.8 1.8) (layer B.CrtYd) (width 0.05))
+    (fp_line (start -1.8 -6.85) (end 1.8 -6.85) (layer B.CrtYd) (width 0.05))
+    (fp_line (start -1.8 1.8) (end -1.8 -6.85) (layer B.CrtYd) (width 0.05))
+    (fp_line (start -1.33 1.33) (end 0 1.33) (layer B.SilkS) (width 0.12))
+    (fp_line (start -1.33 0) (end -1.33 1.33) (layer B.SilkS) (width 0.12))
+    (fp_line (start -1.33 -1.27) (end 1.33 -1.27) (layer B.SilkS) (width 0.12))
+    (fp_line (start 1.33 -1.27) (end 1.33 -6.41) (layer B.SilkS) (width 0.12))
+    (fp_line (start -1.33 -1.27) (end -1.33 -6.41) (layer B.SilkS) (width 0.12))
+    (fp_line (start -1.33 -6.41) (end 1.33 -6.41) (layer B.SilkS) (width 0.12))
+    (fp_line (start -1.27 0.635) (end -0.635 1.27) (layer B.Fab) (width 0.1))
+    (fp_line (start -1.27 -6.35) (end -1.27 0.635) (layer B.Fab) (width 0.1))
+    (fp_line (start 1.27 -6.35) (end -1.27 -6.35) (layer B.Fab) (width 0.1))
+    (fp_line (start 1.27 1.27) (end 1.27 -6.35) (layer B.Fab) (width 0.1))
     (fp_line (start -0.635 1.27) (end 1.27 1.27) (layer B.Fab) (width 0.1))
-    (fp_line (start 1.27 1.27) (end 1.27 -6.35) (layer B.Fab) (width 0.1))
-    (fp_line (start 1.27 -6.35) (end -1.27 -6.35) (layer B.Fab) (width 0.1))
-    (fp_line (start -1.27 -6.35) (end -1.27 0.635) (layer B.Fab) (width 0.1))
-    (fp_line (start -1.27 0.635) (end -0.635 1.27) (layer B.Fab) (width 0.1))
-    (fp_line (start -1.33 -6.41) (end 1.33 -6.41) (layer B.SilkS) (width 0.12))
-    (fp_line (start -1.33 -1.27) (end -1.33 -6.41) (layer B.SilkS) (width 0.12))
-    (fp_line (start 1.33 -1.27) (end 1.33 -6.41) (layer B.SilkS) (width 0.12))
-    (fp_line (start -1.33 -1.27) (end 1.33 -1.27) (layer B.SilkS) (width 0.12))
-    (fp_line (start -1.33 0) (end -1.33 1.33) (layer B.SilkS) (width 0.12))
-    (fp_line (start -1.33 1.33) (end 0 1.33) (layer B.SilkS) (width 0.12))
-    (fp_line (start -1.8 1.8) (end -1.8 -6.85) (layer B.CrtYd) (width 0.05))
-    (fp_line (start -1.8 -6.85) (end 1.8 -6.85) (layer B.CrtYd) (width 0.05))
-    (fp_line (start 1.8 -6.85) (end 1.8 1.8) (layer B.CrtYd) (width 0.05))
-    (fp_line (start 1.8 1.8) (end -1.8 1.8) (layer B.CrtYd) (width 0.05))
     (fp_text user %R (at 0 -2.54 270) (layer B.Fab)
       (effects (font (size 1 1) (thickness 0.15)) (justify mirror))
@@
       (effects (font (size 1 1) (thickness 0.15)) (justify mirror))
     )
+    (fp_line (start 1.8 1.8) (end -1.8 1.8) (layer B.CrtYd) (width 0.05))
+    (fp_line (start 1.8 -6.85) (end 1.8 1.8) (layer B.CrtYd) (width 0.05))
+    (fp_line (start -1.8 -6.85) (end 1.8 -6.85) (layer B.CrtYd) (width 0.05))
+    (fp_line (start -1.8 1.8) (end -1.8 -6.85) (layer B.CrtYd) (width 0.05))
+    (fp_line (start -1.33 1.33) (end 0 1.33) (layer B.SilkS) (width 0.12))
+    (fp_line (start -1.33 0) (end -1.33 1.33) (layer B.SilkS) (width 0.12))
+    (fp_line (start -1.33 -1.27) (end 1.33 -1.27) (layer B.SilkS) (width 0.12))
+    (fp_line (start 1.33 -1.27) (end 1.33 -6.41) (layer B.SilkS) (width 0.12))
+    (fp_line (start -1.33 -1.27) (end -1.33 -6.41) (layer B.SilkS) (width 0.12))
+    (fp_line (start -1.33 -6.41) (end 1.33 -6.41) (layer B.SilkS) (width 0.12))
+    (fp_line (start -1.27 0.635) (end -0.635 1.27) (layer B.Fab) (width 0.1))
+    (fp_line (start -1.27 -6.35) (end -1.27 0.635) (layer B.Fab) (width 0.1))
+    (fp_line (start 1.27 -6.35) (end -1.27 -6.35) (layer B.Fab) (width 0.1))
+    (fp_line (start 1.27 1.27) (end 1.27 -6.35) (layer B.Fab) (width 0.1))
     (fp_line (start -0.635 1.27) (end 1.27 1.27) (layer B.Fab) (width 0.1))
-    (fp_line (start 1.27 1.27) (end 1.27 -6.35) (layer B.Fab) (width 0.1))
-    (fp_line (start 1.27 -6.35) (end -1.27 -6.35) (layer B.Fab) (width 0.1))
-    (fp_line (start -1.27 -6.35) (end -1.27 0.635) (layer B.Fab) (width 0.1))
-    (fp_line (start -1.27 0.635) (end -0.635 1.27) (layer B.Fab) (width 0.1))
-    (fp_line (start -1.33 -6.41) (end 1.33 -6.41) (layer B.SilkS) (width 0.12))
-    (fp_line (start -1.33 -1.27) (end -1.33 -6.41) (layer B.SilkS) (width 0.12))
-    (fp_line (start 1.33 -1.27) (end 1.33 -6.41) (layer B.SilkS) (width 0.12))
-    (fp_line (start -1.33 -1.27) (end 1.33 -1.27) (layer B.SilkS) (width 0.12))
-    (fp_line (start -1.33 0) (end -1.33 1.33) (layer B.SilkS) (width 0.12))
-    (fp_line (start -1.33 1.33) (end 0 1.33) (layer B.SilkS) (width 0.12))
-    (fp_line (start -1.8 1.8) (end -1.8 -6.85) (layer B.CrtYd) (width 0.05))
-    (fp_line (start -1.8 -6.85) (end 1.8 -6.85) (layer B.CrtYd) (width 0.05))
-    (fp_line (start 1.8 -6.85) (end 1.8 1.8) (layer B.CrtYd) (width 0.05))
-    (fp_line (start 1.8 1.8) (end -1.8 1.8) (layer B.CrtYd) (width 0.05))
     (fp_text user %R (at 0 -2.54 270) (layer B.Fab)
       (effects (font (size 1 1) (thickness 0.15)) (justify mirror))
@@
     (effects (font (size 0.5 0.5) (thickness 0.075)) (justify mirror))
   )
-  (gr_text "breadled\nv0.2" (at 153.035 83.82 90) (layer B.SilkS)
+  (gr_text "breadled\nv0.2.1" (at 153.035 83.82 90) (layer B.SilkS)
     (effects (font (size 0.5 0.5) (thickness 0.075)) (justify right mirror))
   )
@@
   (segment (start 149.86 83.82) (end 151.062081 83.82) (width 1) (layer F.Cu) (net 2))
   (segment (start 155.36 81.28) (end 155.27 81.37) (width 1) (layer F.Cu) (net 3))
+  (segment (start 157.39 81.37) (end 157.48 81.28) (width 1) (layer F.Cu) (net 3))
+  (segment (start 155.27 81.37) (end 157.39 81.37) (width 1) (layer F.Cu) (net 3))
+  (segment (start 149.86 81.28) (end 157.48 81.28) (width 1) (layer B.Cu) (net 3))
   (segment (start 151.98 86.36) (end 152.07 86.27) (width 1) (layer F.Cu) (net 4))
   (segment (start 149.86 86.36) (end 151.98 86.36) (width 1) (layer F.Cu) (net 4))
